Commit message: feat: switch retargeting to HKU vector IK

File: assets/mmhand/urdf/hand.urdf (robot description, URDF)
Before this commit: robot mmhand, 27 links, 26 joints
Links:
- removed link finger_1_distal_phalanx_1
- removed link finger_1_fingertip_1
- removed link finger_1_proximal_phalanx_1
- removed link finger_2_distal_phalanx_1
- removed link finger_2_fingertip_1
- removed link finger_2_proximal_phalanx_1
- removed link finger_3_distal_phalanx_1
- removed link finger_3_fingertip_1
- removed link finger_3_proximal_phalanx_1
- removed link finger_4_distal_phalanx_1
- removed link finger_4_fingertip_1
- removed link finger_4_proximal_phalanx_1
- removed link mmhand_thumb_1_finger_7_distal_phalanx_1
- removed link mmhand_thumb_1_finger_7_fingertip_1
- removed link mmhand_thumb_1_finger_7_proximal_phalanx_1
- removed link mmhand_thumb_1_thumb_abduction_adduction_link_1
- removed link mmhand_thumb_1_thumb_base_1
- removed link palm_1
- removed link palm_1_abduction_adduction_link_1
- removed link palm_1_abduction_adduction_link_2
- removed link palm_1_abduction_adduction_link_3
- removed link palm_1_abduction_adduction_link_4
- removed link palm_1_finger_base_1
- removed link palm_1_finger_base_2
- removed link palm_1_finger_base_3
- removed link palm_1_finger_base_4
- added link 1-1_Link, mass 0.00230230069636072; collision mesh filename=../meshes/1-1_Link.STL; visual mesh filename=../meshes/1-1_Link.STL
- added link 1-2_Link, mass 0.00692845319857682; collision mesh filename=../meshes/1-2_Link.STL; visual mesh filename=../meshes/1-2_Link.STL
- added link 1-3_Link, mass 0.0069931373751404; collision mesh filename=../meshes/1-3_Link.STL; visual mesh filename=../meshes/1-3_Link.STL
- added link 1-4_Link, mass 0.00512412476728691; collision mesh filename=../meshes/1-4_Link.STL; visual mesh filename=../meshes/1-4_Link.STL
- added link 1-tip_Link
- added link 2-1_Link, mass 0.00230230069636073; collision mesh filename=../meshes/2-1_Link.STL; visual mesh filename=../meshes/2-1_Link.STL
- added link 2-2_Link, mass 0.00712441800265096; collision mesh filename=../meshes/2-2_Link.STL; visual mesh filename=../meshes/2-2_Link.STL
- added link 2-3_Link, mass 0.00725239796486435; collision mesh filename=../meshes/2-3_Link.STL; visual mesh filename=../meshes/2-3_Link.STL
- added link 2-4_Link, mass 0.00512412473433074; collision mesh filename=../meshes/2-4_Link.STL; visual mesh filename=../meshes/2-4_Link.STL
- added link 2-tip_Link
- added link 3-1_Link, mass 0.00230230069636072; collision mesh filename=../meshes/3-1_Link.STL; visual mesh filename=../meshes/3-1_Link.STL
- added link 3-2_Link, mass 0.00692845433306354; collision mesh filename=../meshes/3-2_Link.STL; visual mesh filename=../meshes/3-2_Link.STL
- added link 3-3_Link, mass 0.00725239756221735; collision mesh filename=../meshes/3-3_Link.STL; visual mesh filename=../meshes/3-3_Link.STL
- added link 3-4_Link, mass 0.00512413487399222; collision mesh filename=../meshes/3-4_Link.STL; visual mesh filename=../meshes/3-4_Link.STL
- added link 3-tip_Link
- added link 4-1_Link, mass 0.00230230069636074; collision mesh filename=../meshes/4-1_Link.STL; visual mesh filename=../meshes/4-1_Link.STL
- added link 4-2_Link, mass 0.00481072140661494; collision mesh filename=../meshes/4-2_Link.STL; visual mesh filename=../meshes/4-2_Link.STL
- added link 4-3_Link, mass 0.00725239796482652; collision mesh filename=../meshes/4-3_Link.STL; visual mesh filename=../meshes/4-3_Link.STL
- added link 4-4_Link, mass 0.00512412742148302; collision mesh filename=../meshes/4-4_Link.STL; visual mesh filename=../meshes/4-4_Link.STL
- added link 4-tip_Link
- added link 5-1_Link, mass 0.0132709127980221; collision mesh filename=../meshes/5-1_Link.STL; visual mesh filename=../meshes/5-1_Link.STL
- added link 5-2_Link, mass 0.00220880787835431; collision mesh filename=../meshes/5-2_Link.STL; visual mesh filename=../meshes/5-2_Link.STL
- added link 5-3_Link, mass 0.00712436486474142; collision mesh filename=../meshes/5-3_Link.STL; visual mesh filename=../meshes/5-3_Link.STL
- added link 5-4_Link, mass 0.00725239164238573; collision mesh filename=../meshes/5-4_Link.STL; visual mesh filename=../meshes/5-4_Link.STL
- added link 5-5_Link, mass 0.00512406201240643; collision mesh filename=../meshes/5-5_Link.STL; visual mesh filename=../meshes/5-5_Link.STL
- added link 5-tip_Link
- link base_link: mass 0.07274593771183077 -> 0.19106535154014; geometry collision mesh filename=../meshes/base_link.STL; visual mesh filename=../meshes/base_link.STL
Joints:
- removed joint index_aa_joint
- removed joint little_aa_joint
- removed joint middle_aa_joint
- removed joint mmhand_finger_1_distal_phalanx_1_pip_joint
- removed joint mmhand_finger_1_fingertip_1_dip_joint
- removed joint mmhand_finger_1_proximal_phalanx_1_mcp_fe_joint
- removed joint mmhand_finger_2_distal_phalanx_1_pip_joint
- removed joint mmhand_finger_2_fingertip_1_dip_joint
- removed joint mmhand_finger_2_proximal_phalanx_1_mcp_fe_joint
- removed joint mmhand_finger_3_distal_phalanx_1_pip_joint
- removed joint mmhand_finger_3_fingertip_1_dip_joint
- removed joint mmhand_finger_3_proximal_phalanx_1_mcp_fe_joint
- removed joint mmhand_finger_4_distal_phalanx_1_pip_joint
- removed joint mmhand_finger_4_fingertip_1_dip_joint
- removed joint mmhand_finger_4_proximal_phalanx_1_mcp_fe_joint
- removed joint mmhand_thumb_1_mmhand_finger_5_distal_phalanx_1_pip_joint
- removed joint mmhand_thumb_1_mmhand_finger_5_fingertip_1_dip_joint
- removed joint mmhand_thumb_1_mmhand_finger_5_proximal_phalanx_1_mcp_fe_joint
- removed joint palm_1_finger_base_1_fixed_joint
- removed joint palm_1_finger_base_2_fixed_joint
- removed joint palm_1_finger_base_3_fixed_joint
- removed joint palm_1_finger_base_4_fixed_joint
- removed joint palm_1_fixed_joint
- removed joint ring_aa_joint
- removed joint thumb_aa_joint
- removed joint thumb_cmc1_joint
- added joint 1-1: type revolute, parent base_link, child 1-1_Link, origin xyz=0.097499 -0.025791 0.0074875 rpy=0 0 0, axis 0 0 1, limit lower=-0.8727 upper=0.5236 effort=0 velocity=0
- added joint 1-2: type revolute, parent 1-1_Link, child 1-2_Link, origin xyz=0.012725 0 -0.0014425 rpy=-1.5708 -0.029375 0, axis 0 0 1, limit lower=0 upper=1.5708 effort=0 velocity=0
- added joint 1-3: type revolute, parent 1-2_Link, child 1-3_Link, origin xyz=0.035 0 0.0001495 rpy=0 0 0.024907, axis 0 0 1, limit lower=0 upper=1.4835 effort=0 velocity=0
- added joint 1-4: type revolute, parent 1-3_Link, child 1-4_Link, origin xyz=0.028 0 -0.00029976 rpy=0 0 -0.00068633, axis 0 0 1, limit lower=0 upper=1.5708 effort=0 velocity=0
- added joint 1-tip: type fixed, parent 1-4_Link, child 1-tip_Link, origin xyz=0.022 0 0 rpy=0 0 0
- added joint 2-1: type revolute, parent base_link, child 2-1_Link, origin xyz=0.1025 -0.0017912 0.0074875 rpy=0 0 0, axis 0 0 1, limit lower=-0.8727 upper=0.8727 effort=0 velocity=0
- added joint 2-2: type revolute, parent 2-1_Link, child 2-2_Link, origin xyz=0.012725 0 -0.0014425 rpy=-1.5708 0 0, axis 0 0 1, limit lower=0 upper=1.5708 effort=0 velocity=0
- added joint 2-3: type revolute, parent 2-2_Link, child 2-3_Link, origin xyz=0.034985 -0.0010281 0.0001495 rpy=0 0 0, axis 0 0 1, limit lower=0 upper=1.4835 effort=0 velocity=0
- added joint 2-4: type revolute, parent 2-3_Link, child 2-4_Link, origin xyz=0.028 -0.00012529 -0.00029976 rpy=0 0 0, axis 0 0 1, limit lower=0 upper=1.5708 effort=0 velocity=0
- added joint 2-tip: type fixed, parent 2-4_Link, child 2-tip_Link, origin xyz=0.022 0 0 rpy=0 0 0
- added joint 3-1: type revolute, parent base_link, child 3-1_Link, origin xyz=0.097499 0.022209 0.0074875 rpy=0 0 0, axis 0 0 1, limit lower=-0.5236 upper=1.1345 effort=0 velocity=0
- added joint 3-2: type revolute, parent 3-1_Link, child 3-2_Link, origin xyz=0.012725 0 -0.0014425 rpy=-1.5708 0 0, axis 0 0 1, limit lower=0 upper=1.5708 effort=0 velocity=0
- added joint 3-3: type revolute, parent 3-2_Link, child 3-3_Link, origin xyz=0.034999 0.00019049 0.0001495 rpy=0 0 0, axis 0 0 1, limit lower=0 upper=1.4835 effort=0 velocity=0
- added joint 3-4: type revolute, parent 3-3_Link, child 3-4_Link, origin xyz=0.027987 0.00084958 -0.00029976 rpy=0 0 0, axis 0 0 1, limit lower=0 upper=1.5708 effort=0 velocity=0
- added joint 3-tip: type fixed, parent 3-4_Link, child 3-tip_Link, origin xyz=0.022 0 0 rpy=0 0 0
- added joint 4-1: type revolute, parent base_link, child 4-1_Link, origin xyz=0.081999 0.046209 0.0074875 rpy=0 0 0, axis 0 0 1, limit lower=-0.3491 upper=1.1345 effort=0 velocity=0
- added joint 4-2: type revolute, parent 4-1_Link, child 4-2_Link, origin xyz=0.012725 0 -0.0014425 rpy=-1.5708 0 0, axis 0 0 1, limit lower=0 upper=1.5708 effort=0 velocity=0
- added joint 4-3: type revolute, parent 4-2_Link, child 4-3_Link, origin xyz=0.034985 -0.0010281 0.0001495 rpy=0 0 0, axis 0 0 1, limit lower=0 upper=1.4835 effort=0 velocity=0
- added joint 4-4: type revolute, parent 4-3_Link, child 4-4_Link, origin xyz=0.028 -0.00012529 -0.00029976 rpy=0 0 0, axis 0 0 1, limit lower=0 upper=1.5708 effort=0 velocity=0
- added joint 4-tip: type fixed, parent 4-4_Link, child 4-tip_Link, origin xyz=0.022 0 0 rpy=0 0 0
- added joint 5-1: type revolute, parent base_link, child 5-1_Link, origin xyz=0.036402 -0.026652 0.010947 rpy=0 0 -2.3951, axis 0 0 1, limit lower=-1.0308 upper=0.5400 effort=0 velocity=0
- added joint 5-2: type revolute, parent 5-1_Link, child 5-2_Link, origin xyz=0.0016159 0.0014636 -0.035499 rpy=0.73235 1.0562 0.78487, axis 0 0 1, limit lower=-1.0472 upper=1.0472 effort=0 velocity=0
- added joint 5-3: type revolute, parent 5-2_Link, child 5-3_Link, origin xyz=0.012725 0 -0.0014425 rpy=-1.5708 0.47834 0, axis 0 0 1, limit lower=0 upper=1.5708 effort=0 velocity=0
- added joint 5-4: type revolute, parent 5-3_Link, child 5-4_Link, origin xyz=0.035 0 0.0001495 rpy=0 0 0.19193, axis 0 0 1, limit lower=0 upper=1.4835 effort=0 velocity=0
- added joint 5-5: type revolute, parent 5-4_Link, child 5-5_Link, origin xyz=0.02761 -0.0046551 -0.00029976 rpy=0 0 0, axis 0 0 1, limit lower=0 upper=1.5708 effort=0 velocity=0
- added joint 5-tip: type fixed, parent 5-5_Link, child 5-tip_Link, origin xyz=0.020 0 0 rpy=0 0 0
