Commit message: replace retarget model with current mmhand urdf

File: assets/mmhand/urdf/hand.urdf (robot description, URDF)
Before this commit: robot HKU Hand, 27 links, 26 joints
Links:
- removed link 1-1_Link
- removed link 1-2_Link
- removed link 1-3_Link
- removed link 1-4_Link
- removed link 2-1_Link
- removed link 2-2_Link
- removed link 2-3_Link
- removed link 2-4_Link
- removed link 3-1_Link
- removed link 3-2_Link
- removed link 3-3_Link
- removed link 3-4_Link
- removed link 4-1_Link
- removed link 4-2_Link
- removed link 4-3_Link
- removed link 4-4_Link
- removed link 5-1_Link
- removed link 5-2_Link
- removed link 5-3_Link
- removed link 5-4_Link
- removed link 5-5_Link
- added link finger_1_distal_phalanx_1, mass 0.006680553833901148; collision cylinder length=0.021502949 radius=0.009876129; collision sphere radius=0.009876129
- added link finger_1_fingertip_1, mass 0.005701382551402315; collision cylinder length=0.020835574 radius=0.009262807; collision sphere radius=0.009262807
- added link finger_1_proximal_phalanx_1, mass 0.008314052389766543; collision cylinder length=0.026569046 radius=0.012400477; collision sphere radius=0.012400477
- added link finger_2_distal_phalanx_1, mass 0.006680553833901148; collision cylinder length=0.021361511 radius=0.009953366; collision sphere radius=0.009953366
- added link finger_2_fingertip_1, mass 0.005701382551402315; collision cylinder length=0.020857118 radius=0.009286031; collision sphere radius=0.009286031
- added link finger_2_proximal_phalanx_1, mass 0.008314052389766543; collision cylinder length=0.02647651 radius=0.012424022; collision sphere radius=0.012424022
- added link finger_3_distal_phalanx_1, mass 0.006680553833901148; collision cylinder length=0.021533148 radius=0.009870392; collision sphere radius=0.009870392
- added link finger_3_fingertip_1, mass 0.005701382551402315; collision cylinder length=0.020924213 radius=0.009249611; collision sphere radius=0.009249611
- added link finger_3_proximal_phalanx_1, mass 0.008314052389766543; collision cylinder length=0.026506101 radius=0.012421897; collision sphere radius=0.012421897
- added link finger_4_distal_phalanx_1, mass 0.006680553833901148; collision cylinder length=0.021533255 radius=0.009870318; collision sphere radius=0.009870318
- added link finger_4_fingertip_1, mass 0.005701382551402315; collision cylinder length=0.020924206 radius=0.009249611; collision sphere radius=0.009249611
- added link finger_4_proximal_phalanx_1, mass 0.008314052389766543; collision cylinder length=0.026506104 radius=0.012421896; collision sphere radius=0.012421896
- added link mmhand_thumb_1_finger_7_distal_phalanx_1, mass 0.006680553833901148; collision cylinder length=0.021416021 radius=0.009876707; collision sphere radius=0.009876707
- added link mmhand_thumb_1_finger_7_fingertip_1, mass 0.005701382551402315; collision cylinder length=0.020825109 radius=0.00930797; collision sphere radius=0.00930797
- added link mmhand_thumb_1_finger_7_proximal_phalanx_1, mass 0.008314052389766543; collision cylinder length=0.026566819 radius=0.012435313; collision sphere radius=0.012435313
- added link mmhand_thumb_1_thumb_abduction_adduction_link_1, mass 0.0037666395780571542; collision mesh filename=../meshes/mmhand_thumb_1_thumb_abduction_adduction_link_1.s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 scale=0.001 0.001 0.001; visual mesh filename=../meshes/mmhand_thumb_1_thumb_abduction_adduction_link_1.s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 scale=0.001 0.001 0.001
- added link mmhand_thumb_1_thumb_base_1, mass 0.01857949246514449; collision mesh filename=../meshes/mmhand_thumb_1_thumb_base_1.stl scale=0.001 0.001 0.001; visual mesh filename=../meshes/mmhand_thumb_1_thumb_base_1.stl scale=0.001 0.001 0.001
- added link palm_1, mass 0.16539031129630477; collision mesh filename=../meshes/palm_1.stl scale=0.001 0.001 0.001; visual mesh filename=../meshes/palm_1.stl scale=0.001 0.001 0.001
- added link palm_1_abduction_adduction_link_1, mass 0.0038835140540164664; collision mesh filename=../meshes/palm_1_abduction_adduction_link_1.stl scale=0.001 0.001 0.001; visual mesh filename=../meshes/palm_1_abduction_adduction_link_1.stl scale=0.001 0.001 0.001
- added link palm_1_abduction_adduction_link_2, mass 0.0038835140540164664; collision mesh filename=../meshes/palm_1_abduction_adduction_link_2.stl scale=0.001 0.001 0.001; visual mesh filename=../meshes/palm_1_abduction_adduction_link_2.stl scale=0.001 0.001 0.001
- added link palm_1_abduction_adduction_link_3, mass 0.0038835140540164664; collision mesh filename=../meshes/palm_1_abduction_adduction_link_3.stl scale=0.001 0.001 0.001; visual mesh filename=../meshes/palm_1_abduction_adduction_link_3.stl scale=0.001 0.001 0.001
- added link palm_1_abduction_adduction_link_4, mass 0.0038835140540164664; collision mesh filename=../meshes/palm_1_abduction_adduction_link_4.stl scale=0.001 0.001 0.001; visual mesh filename=../meshes/palm_1_abduction_adduction_link_4.stl scale=0.001 0.001 0.001
- added link palm_1_finger_base_1, mass 0.010915583239628221; collision mesh filename=../meshes/palm_1_finger_base_1.stl scale=0.001 0.001 0.001; visual mesh filename=../meshes/palm_1_finger_base_1.stl scale=0.001 0.001 0.001
- added link palm_1_finger_base_2, mass 0.010915583239628221; collision mesh filename=../meshes/palm_1_finger_base_2.stl scale=0.001 0.001 0.001; visual mesh filename=../meshes/palm_1_finger_base_2.stl scale=0.001 0.001 0.001
- added link palm_1_finger_base_3, mass 0.010915583239628221; collision mesh filename=../meshes/palm_1_finger_base_3.stl scale=0.001 0.001 0.001; visual mesh filename=../meshes/palm_1_finger_base_3.stl scale=0.001 0.001 0.001
- added link palm_1_finger_base_4, mass 0.010915583239628221; collision mesh filename=../meshes/palm_1_finger_base_4.stl scale=0.001 0.001 0.001; visual mesh filename=../meshes/palm_1_finger_base_4.stl scale=0.001 0.001 0.001
- link base_link: mass 0.19106535154014 -> 0.026671469266356558; geometry collision mesh filename=../meshes/base_link.stl scale=0.001 0.001 0.001; visual mesh filename=../meshes/base_link.stl scale=0.001 0.001 0.001
Joints:
- removed joint 1-1
- removed joint 1-2
- removed joint 1-3
- removed joint 1-4
- removed joint 2-1
- removed joint 2-2
- removed joint 2-3
- removed joint 2-4
- removed joint 3-1
- removed joint 3-2
- removed joint 3-3
- removed joint 3-4
- removed joint 4-1
- removed joint 4-2
- removed joint 4-3
- removed joint 4-4
- removed joint 5-1
- removed joint 5-2
- removed joint 5-3
- removed joint 5-4
- removed joint 5-5
- added joint Index_MCP_AA: type revolute, parent palm_1_finger_base_1, child palm_1_abduction_adduction_link_1, origin xyz=0.098962 -0.040332 -0.023497 rpy=0.0 -0.0 0.0, axis -0.0 0.0 -1.0, limit lower=0.0 upper=1.012291 effort=100 velocity=100
- added joint Index_MCP_FE: type revolute, parent palm_1_abduction_adduction_link_1, child finger_1_proximal_phalanx_1, origin xyz=0.011655 0.00511 -0.0114 rpy=0.0 -0.0 0.0, axis -0.390731 0.920505 -0.0, limit lower=-0.244346 upper=1.570796 effort=100 velocity=100
- added joint Little_MCP_AA: type revolute, parent palm_1_finger_base_4, child palm_1_abduction_adduction_link_4, origin xyz=0.098962 -0.040332 -0.023497 rpy=0.0 -0.0 0.0, axis -0.0 -0.0 -1.0, limit lower=0.0 upper=0.942478 effort=100 velocity=100
- added joint Little_MCP_FE: type revolute, parent palm_1_abduction_adduction_link_4, child finger_4_proximal_phalanx_1, origin xyz=0.010207 0.007601 -0.0114 rpy=0.0 -0.0 0.0, axis -0.587785 0.809017 0.0, limit lower=-0.261799 upper=1.570796 effort=100 velocity=100
- added joint Middle_MCP_AA: type revolute, parent palm_1_finger_base_2, child palm_1_abduction_adduction_link_2, origin xyz=0.098962 -0.040332 -0.023497 rpy=0.0 -0.0 0.0, axis -0.0 0.0 -1.0, limit lower=0.0 upper=1.029744 effort=100 velocity=100
- added joint Middle_MCP_FE: type revolute, parent palm_1_abduction_adduction_link_2, child finger_2_proximal_phalanx_1, origin xyz=0.01083 0.006683 -0.0114 rpy=0.0 -0.0 0.0, axis -0.515038 0.857167 -0.0, limit lower=-0.244346 upper=1.570796 effort=100 velocity=100
- added joint Ring_MCP_AA: type revolute, parent palm_1_finger_base_3, child palm_1_abduction_adduction_link_3, origin xyz=0.098962 -0.040332 -0.023497 rpy=0.0 -0.0 0.0, axis -0.0 -0.0 -1.0, limit lower=0.0 upper=1.064651 effort=100 velocity=100
- added joint Ring_MCP_FE: type revolute, parent palm_1_abduction_adduction_link_3, child finger_3_proximal_phalanx_1, origin xyz=0.010207 0.007601 -0.0114 rpy=0.0 -0.0 0.0, axis -0.587785 0.809017 0.0, limit lower=-0.261799 upper=1.570796 effort=100 velocity=100
- added joint Thumb_CMC: type revolute, parent palm_1, child mmhand_thumb_1_thumb_base_1, origin xyz=-0.052098 -0.000861 0.0088 rpy=0.0 -0.0 0.0, axis 0.0 0.0 -1.0, limit lower=0.0 upper=1.343904 effort=100 velocity=100
- added joint Thumb_MCP_AA: type revolute, parent mmhand_thumb_1_thumb_base_1, child mmhand_thumb_1_thumb_abduction_adduction_link_1, origin xyz=0.000906 -0.012002 -0.045452 rpy=0.0 -0.0 0.0, axis -0.070801 0.928071 -0.365612, limit lower=0.0 upper=0.994838 effort=100 velocity=100
- added joint Thumb_MCP_FE: type revolute, parent mmhand_thumb_1_thumb_abduction_adduction_link_1, child mmhand_thumb_1_finger_7_proximal_phalanx_1, origin xyz=0.005694 0.007003 -0.014507 rpy=0.0 -0.0 0.0, axis 0.862725 0.240955 0.444574, limit lower=-0.331613 upper=1.570796 effort=100 velocity=100
- added joint finger_1_distal_phalanx_1_PIP_Joint: type revolute, parent finger_1_proximal_phalanx_1, child finger_1_distal_phalanx_1, origin xyz=0.036074 0.015166 -6e-05 rpy=0.0 -0.0 0.0, axis -0.390731 0.920505 -0.0, limit lower=-0.15708 upper=1.553343 effort=100 velocity=100
- added joint finger_1_fingertip_1_DIP_Joint: type revolute, parent finger_1_distal_phalanx_1, child finger_1_fingertip_1, origin xyz=0.028369 0.007387 -5e-06 rpy=0.0 -0.0 0.0, axis -0.390731 0.920505 -0.0, limit lower=-0.226893 upper=1.762783 effort=100 velocity=100
- added joint finger_2_distal_phalanx_1_PIP_Joint: type revolute, parent finger_2_proximal_phalanx_1, child finger_2_distal_phalanx_1, origin xyz=0.033613 0.020039 -6e-05 rpy=0.0 -0.0 0.0, axis -0.515038 0.857167 -0.0, limit lower=-0.15708 upper=1.553343 effort=100 velocity=100
- added joint finger_2_fingertip_1_DIP_Joint: type revolute, parent finger_2_distal_phalanx_1, child finger_2_fingertip_1, origin xyz=0.027065 0.011263 -5e-06 rpy=0.0 -0.0 0.0, axis -0.515038 0.857167 -0.0, limit lower=-0.226893 upper=1.762783 effort=100 velocity=100
- added joint finger_3_distal_phalanx_1_PIP_Joint: type revolute, parent finger_3_proximal_phalanx_1, child finger_3_distal_phalanx_1, origin xyz=0.031738 0.022892 -6e-05 rpy=0.0 -0.0 0.0, axis -0.587785 0.809017 0.0, limit lower=-0.15708 upper=1.553343 effort=100 velocity=100
- added joint finger_3_fingertip_1_DIP_Joint: type revolute, parent finger_3_distal_phalanx_1, child finger_3_fingertip_1, origin xyz=0.02598 0.013579 -5e-06 rpy=0.0 -0.0 0.0, axis -0.587785 0.809017 -0.0, limit lower=-0.226893 upper=1.762783 effort=100 velocity=100
- added joint finger_4_distal_phalanx_1_PIP_Joint: type revolute, parent finger_4_proximal_phalanx_1, child finger_4_distal_phalanx_1, origin xyz=0.031738 0.022892 -6e-05 rpy=0.0 -0.0 0.0, axis -0.587785 0.809017 0.0, limit lower=-0.15708 upper=1.553343 effort=100 velocity=100
- added joint finger_4_fingertip_1_DIP_Joint: type revolute, parent finger_4_distal_phalanx_1, child finger_4_fingertip_1, origin xyz=0.02598 0.013579 -5e-06 rpy=0.0 -0.0 0.0, axis -0.587785 0.809017 -0.0, limit lower=-0.226893 upper=1.762783 effort=100 velocity=100
- added joint mmhand_thumb_1_finger_7_distal_phalanx_1_PIP_Joint: type revolute, parent mmhand_thumb_1_finger_7_proximal_phalanx_1, child mmhand_thumb_1_finger_7_distal_phalanx_1, origin xyz=0.019099 -0.007442 -0.033335 rpy=0.0 -0.0 0.0, axis 0.862725 0.240955 0.444574, limit lower=-0.15708 upper=1.553343 effort=100 velocity=100
- added joint mmhand_thumb_1_finger_7_fingertip_1_DIP_Joint: type revolute, parent mmhand_thumb_1_finger_7_distal_phalanx_1, child mmhand_thumb_1_finger_7_fingertip_1, origin xyz=0.010549 -0.006561 -0.026553 rpy=0.0 -0.0 0.0, axis 0.862725 0.240955 0.444574, limit lower=-0.226893 upper=1.762783 effort=100 velocity=100
- added joint palm_1_finger_base_1_fixed_joint: type fixed, parent palm_1, child palm_1_finger_base_1, origin xyz=-0.1039 0.040332 0.023697 rpy=0.0 -0.0 0.0
- added joint palm_1_finger_base_2_fixed_joint: type fixed, parent palm_1, child palm_1_finger_base_2, origin xyz=-0.1036 0.064332 0.023697 rpy=0.0 -0.0 0.0
- added joint palm_1_finger_base_3_fixed_joint: type fixed, parent palm_1, child palm_1_finger_base_3, origin xyz=-0.1039 0.088332 0.023697 rpy=0.0 -0.0 0.0
- added joint palm_1_finger_base_4_fixed_joint: type fixed, parent palm_1, child palm_1_finger_base_4, origin xyz=-0.119644 0.112222 0.023665 rpy=0.0 -0.0 0.0
- added joint palm_1_fixed_joint: type fixed, parent base_link, child palm_1, origin xyz=0.099 -0.040324 -0.033543 rpy=0.0 -0.0 0.0
- joint 1-tip: origin xyz=0.022 0 0 rpy=0 0 0 -> xyz=0.023001459 0.010424364 -0.004367931 rpy=0 0 0; parent 1-4_Link -> finger_1_fingertip_1
- joint 2-tip: origin xyz=0.022 0 0 rpy=0 0 0 -> xyz=0.021343147 0.013505685 -0.004311705 rpy=0 0 0; parent 2-4_Link -> finger_2_fingertip_1
- joint 3-tip: origin xyz=0.022 0 0 rpy=0 0 0 -> xyz=0.020106421 0.015325961 -0.004336191 rpy=0 0 0; parent 3-4_Link -> finger_3_fingertip_1
- joint 4-tip: origin xyz=0.022 0 0 rpy=0 0 0 -> xyz=0.020105907 0.015325727 -0.004336522 rpy=0 0 0; parent 4-4_Link -> finger_4_fingertip_1
- joint 5-tip: origin xyz=0.020 0 0 rpy=0 0 0 -> xyz=0.012366569 -0.000590601 -0.022397383 rpy=0 0 0; parent 5-5_Link -> mmhand_thumb_1_finger_7_fingertip_1

Commit message: 临时调整urdf限位进行实验

File: assets/mmhand/urdf/hand.urdf (robot description, URDF)
Before this commit: robot mmhand, 32 links, 31 joints
Joints:
- joint Thumb_CMC: limit lower=0.0 upper=1.343904 effort=100 velocity=100 -> lower=0.7 upper=1.51 effort=100 velocity=100
- joint Thumb_MCP_AA: limit lower=0.0 upper=0.994838 effort=100 velocity=100 -> lower=-1.2 upper=0.07 effort=100 velocity=100

Commit message: Simplify D435 hand tracking pipeline

File: assets/mmhand/urdf/hand.urdf (robot description, URDF)
Before this commit: robot mmhand, 32 links, 31 joints
Joints:
- joint Index_MCP_AA: limit lower=0.0 upper=1.012291 effort=100 velocity=100 -> lower=-0.134680076 upper=0.683316809 effort=100 velocity=100; origin xyz=0.098962 -0.040332 -0.023497 rpy=0.0 -0.0 0.0 -> xyz=0.098962 -0.040332 -0.023497 rpy=0.168155027 0.104836067 0.000000000
- joint Little_MCP_AA: limit lower=0.0 upper=0.942478 effort=100 velocity=100 -> lower=-0.512305480 upper=0.348147973 effort=100 velocity=100; origin xyz=0.098962 -0.040332 -0.023497 rpy=0.0 -0.0 0.0 -> xyz=0.098962 -0.040332 -0.023497 rpy=-0.117078813 0.071869646 0.000000000
- joint Middle_MCP_AA: limit lower=0.0 upper=1.029744 effort=100 velocity=100 -> lower=-0.083333135 upper=0.456340549 effort=100 velocity=100; origin xyz=0.098962 -0.040332 -0.023497 rpy=0.0 -0.0 0.0 -> xyz=0.098962 -0.040332 -0.023497 rpy=0.074673382 0.123211157 0.000000000
- joint Ring_MCP_AA: limit lower=0.0 upper=1.064651 effort=100 velocity=100 -> lower=-0.128152636 upper=0.518288581 effort=100 velocity=100; origin xyz=0.098962 -0.040332 -0.023497 rpy=0.0 -0.0 0.0 -> xyz=0.098962 -0.040332 -0.023497 rpy=-0.029471042 0.354478058 0.000000000
- joint Thumb_CMC: limit lower=0.7 upper=1.51 effort=100 velocity=100 -> lower=0.814912478 upper=2.149352256 effort=100 velocity=100
- joint Thumb_MCP_AA: limit lower=-1.2 upper=0.07 effort=100 velocity=100 -> lower=-1.100000000 upper=1.000000000 effort=100 velocity=100

Commit message: feat: refine MMHand retargeting and latency

File: assets/mmhand/urdf/hand.urdf (robot description, URDF)
Before this commit: robot mmhand, 32 links, 31 joints
Joints:
- joint Index_MCP_AA: limit lower=-0.134680076 upper=0.683316809 effort=100 velocity=100 -> lower=0.0 upper=1.012291 effort=100 velocity=100; origin xyz=0.098962 -0.040332 -0.023497 rpy=0.168155027 0.104836067 0.000000000 -> xyz=0.098962 -0.040332 -0.023497 rpy=0.0 -0.0 0.0
- joint Little_MCP_AA: limit lower=-0.512305480 upper=0.348147973 effort=100 velocity=100 -> lower=0.0 upper=0.942478 effort=100 velocity=100; origin xyz=0.098962 -0.040332 -0.023497 rpy=-0.117078813 0.071869646 0.000000000 -> xyz=0.098962 -0.040332 -0.023497 rpy=0.0 -0.0 0.0
- joint Middle_MCP_AA: limit lower=-0.083333135 upper=0.456340549 effort=100 velocity=100 -> lower=0.0 upper=1.029744 effort=100 velocity=100; origin xyz=0.098962 -0.040332 -0.023497 rpy=0.074673382 0.123211157 0.000000000 -> xyz=0.098962 -0.040332 -0.023497 rpy=0.0 -0.0 0.0
- joint Ring_MCP_AA: limit lower=-0.128152636 upper=0.518288581 effort=100 velocity=100 -> lower=0.0 upper=1.064651 effort=100 velocity=100; origin xyz=0.098962 -0.040332 -0.023497 rpy=-0.029471042 0.354478058 0.000000000 -> xyz=0.098962 -0.040332 -0.023497 rpy=0.0 -0.0 0.0
- joint Thumb_CMC: limit lower=0.814912478 upper=2.149352256 effort=100 velocity=100 -> lower=0.0 upper=1.343904 effort=100 velocity=100
- joint Thumb_MCP_AA: limit lower=-1.100000000 upper=1.000000000 effort=100 velocity=100 -> lower=0.0 upper=0.994838 effort=100 velocity=100
