Commit message: feat: update MMHand geometry and joint model

File: assets/mmhand/urdf/hand.urdf (robot description, URDF)
Before this commit: robot mmhand, 32 links, 31 joints
Links:
- removed link mmhand_thumb_1_thumb_abduction_adduction_link_1
- removed link palm_1_abduction_adduction_link_4
- removed link palm_1_finger_base_4
- added link mmhand_thumb_1_abduction_adduction_link_without_fin_1, mass 0.0034191812192176027; collision mesh filename=../meshes/mmhand_thumb_1_abduction_adduction_link_without_f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 scale=0.001 0.001 0.001; visual mesh filename=../meshes/mmhand_thumb_1_abduction_adduction_link_without_f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 scale=0.001 0.001 0.001
- added link palm_1_abduction_adduction_link_without_fin_2, mass 0.0034191812192176027; collision mesh filename=../meshes/palm_1_abduction_adduction_link_without_fin_2.stl scale=0.001 0.001 0.001; visual mesh filename=../meshes/palm_1_abduction_adduction_link_without_fin_2.stl scale=0.001 0.001 0.001
- added link palm_1_finger_base_5, mass 0.010861642408655461; collision mesh filename=../meshes/palm_1_finger_base_5.stl scale=0.001 0.001 0.001; visual mesh filename=../meshes/palm_1_finger_base_5.stl scale=0.001 0.001 0.001
- link base_link: mass 0.026671469266356558 -> 0.019420819791017757
- link finger_1_distal_phalanx_1: geometry collision cylinder length=0.021671968 radius=0.009827442; collision sphere radius=0.009827442
- link finger_1_fingertip_1: geometry collision cylinder length=0.020808113 radius=0.009239617; collision sphere radius=0.009239617
- link finger_1_proximal_phalanx_1: mass 0.008314052389766543 -> 0.008314070269239495; geometry collision mesh filename=../meshes/finger_1_proximal_phalanx_1.stl scale=0.001 0.001 0.001; visual mesh filename=../meshes/finger_1_proximal_phalanx_1.stl scale=0.001 0.001 0.001
- link finger_2_distal_phalanx_1: geometry collision cylinder length=0.021671967 radius=0.009827442; collision sphere radius=0.009827442
- link finger_2_fingertip_1: geometry collision cylinder length=0.020808115 radius=0.009239615; collision sphere radius=0.009239615
- link finger_2_proximal_phalanx_1: mass 0.008314052389766543 -> 0.008314070269239495; geometry collision mesh filename=../meshes/finger_2_proximal_phalanx_1.stl scale=0.001 0.001 0.001; visual mesh filename=../meshes/finger_2_proximal_phalanx_1.stl scale=0.001 0.001 0.001
- link finger_3_distal_phalanx_1: geometry collision cylinder length=0.021671968 radius=0.009827442; collision sphere radius=0.009827442
- link finger_3_fingertip_1: geometry collision cylinder length=0.020808112 radius=0.009239617; collision sphere radius=0.009239617
- link finger_3_proximal_phalanx_1: mass 0.008314052389766543 -> 0.008314070269239495; geometry collision mesh filename=../meshes/finger_3_proximal_phalanx_1.stl scale=0.001 0.001 0.001; visual mesh filename=../meshes/finger_3_proximal_phalanx_1.stl scale=0.001 0.001 0.001
- link finger_4_distal_phalanx_1: geometry collision cylinder length=0.021653373 radius=0.009838488; collision sphere radius=0.009838488
- link finger_4_fingertip_1: geometry collision cylinder length=0.020796943 radius=0.009245108; collision sphere radius=0.009245108
- link finger_4_proximal_phalanx_1: mass 0.008314052389766543 -> 0.008314070269239495; geometry collision mesh filename=../meshes/finger_4_proximal_phalanx_1.stl scale=0.001 0.001 0.001; visual mesh filename=../meshes/finger_4_proximal_phalanx_1.stl scale=0.001 0.001 0.001
- link mmhand_thumb_1_finger_7_distal_phalanx_1: geometry collision cylinder length=0.02137981 radius=0.009881072; collision sphere radius=0.009881072
- link mmhand_thumb_1_finger_7_fingertip_1: geometry collision cylinder length=0.020724444 radius=0.009322284; collision sphere radius=0.009322284
- link mmhand_thumb_1_finger_7_proximal_phalanx_1: mass 0.008314052389766543 -> 0.008314070269239495; geometry collision cylinder length=0.026438201 radius=0.012455995; collision sphere radius=0.012455995
- link mmhand_thumb_1_thumb_base_1: mass 0.01857949246514449 -> 0.01870899047965444
- link palm_1: mass 0.16539031129630477 -> 0.6378953328967193
- link palm_1_abduction_adduction_link_1: mass 0.0038835140540164664 -> 0.003787455542299424
- link palm_1_abduction_adduction_link_2: mass 0.0038835140540164664 -> 0.003787455542299424
- link palm_1_abduction_adduction_link_3: mass 0.0038835140540164664 -> 0.003787455542299424
- link palm_1_finger_base_1: mass 0.010915583239628221 -> 0.010861642408655461
- link palm_1_finger_base_2: mass 0.010915583239628221 -> 0.010861642408655461
- link palm_1_finger_base_3: mass 0.010915583239628221 -> 0.010861642408655461
Joints:
- removed joint palm_1_finger_base_4_fixed_joint
- added joint palm_1_finger_base_5_fixed_joint: type fixed, parent palm_1, child palm_1_finger_base_5, origin xyz=-0.117282 0.113474 0.023697 rpy=0.0 -0.0 0.0
- joint Index_MCP_AA: limit lower=0.0 upper=1.012291 effort=100 velocity=100 -> lower=-0.488692 upper=0.628319 effort=100 velocity=100; origin xyz=0.098962 -0.040332 -0.023497 rpy=0.0 -0.0 0.0 -> xyz=0.098962 -0.040332 -0.033397 rpy=0.0 -0.0 0.0
- joint Index_MCP_FE: axis -0.390731 0.920505 -0.0 -> 0.0 1.0 -0.0; origin xyz=0.011655 0.00511 -0.0114 rpy=0.0 -0.0 0.0 -> xyz=0.012725 0.00015 -0.00155 rpy=0.0 -0.0 0.0
- joint Little_MCP_AA: axis -0.0 -0.0 -1.0 -> 0.0 0.0 -1.0; child palm_1_abduction_adduction_link_4 -> palm_1_abduction_adduction_link_without_fin_2; limit lower=0.0 upper=0.942478 effort=100 velocity=100 -> lower=-1.22173 upper=0.366519 effort=100 velocity=100; origin xyz=0.098962 -0.040332 -0.023497 rpy=0.0 -0.0 0.0 -> xyz=0.098962 -0.040335 -0.033397 rpy=0.0 -0.0 0.0; parent palm_1_finger_base_4 -> palm_1_finger_base_5
- joint Little_MCP_FE: axis -0.587785 0.809017 0.0 -> 0.011122 0.999938 -0.0; origin xyz=0.010207 0.007601 -0.0114 rpy=0.0 -0.0 0.0 -> xyz=0.012726 8e-06 -0.001093 rpy=0.0 -0.0 0.0; parent palm_1_abduction_adduction_link_4 -> palm_1_abduction_adduction_link_without_fin_2
- joint Middle_MCP_AA: limit lower=0.0 upper=1.029744 effort=100 velocity=100 -> lower=-0.558505 upper=0.523599 effort=100 velocity=100; origin xyz=0.098962 -0.040332 -0.023497 rpy=0.0 -0.0 0.0 -> xyz=0.098962 -0.040332 -0.033397 rpy=0.0 -0.0 0.0
- joint Middle_MCP_FE: axis -0.515038 0.857167 -0.0 -> 0.0 1.0 -0.0; origin xyz=0.01083 0.006683 -0.0114 rpy=0.0 -0.0 0.0 -> xyz=0.012725 0.00015 -0.00155 rpy=0.0 -0.0 0.0
- joint Ring_MCP_AA: axis -0.0 -0.0 -1.0 -> -0.0 0.0 -1.0; limit lower=0.0 upper=1.064651 effort=100 velocity=100 -> lower=-0.802851 upper=0.453786 effort=100 velocity=100; origin xyz=0.098962 -0.040332 -0.023497 rpy=0.0 -0.0 0.0 -> xyz=0.098962 -0.040332 -0.033397 rpy=0.0 -0.0 0.0
- joint Ring_MCP_FE: axis -0.587785 0.809017 0.0 -> 0.0 1.0 -0.0; origin xyz=0.010207 0.007601 -0.0114 rpy=0.0 -0.0 0.0 -> xyz=0.012725 0.00015 -0.00155 rpy=0.0 -0.0 0.0
- joint Thumb_CMC: limit lower=0.0 upper=1.343904 effort=100 velocity=100 -> lower=0.0 upper=0.942478 effort=100 velocity=100
- joint Thumb_MCP_AA: axis -0.070801 0.928071 -0.365612 -> 0.618416 0.695622 -0.365612; child mmhand_thumb_1_thumb_abduction_adduction_link_1 -> mmhand_thumb_1_abduction_adduction_link_without_fin_1; limit lower=0.0 upper=0.994838 effort=100 velocity=100 -> lower=-1.308997 upper=0.436332 effort=100 velocity=100; origin xyz=0.000906 -0.012002 -0.045452 rpy=0.0 -0.0 0.0 -> xyz=-0.001882 -0.002102 -0.049072 rpy=0.0 -0.0 0.0
- joint Thumb_MCP_FE: axis 0.862725 0.240955 0.444574 -> 0.745353 -0.666627 -0.00761; origin xyz=0.005694 0.007003 -0.014507 rpy=0.0 -0.0 0.0 -> xyz=-0.002098 -0.00243 -0.012412 rpy=0.0 -0.0 0.0; parent mmhand_thumb_1_thumb_abduction_adduction_link_1 -> mmhand_thumb_1_abduction_adduction_link_without_fin_1
- joint finger_1_distal_phalanx_1_PIP_Joint: axis -0.390731 0.920505 -0.0 -> 0.0 1.0 -0.0; origin xyz=0.036074 0.015166 -6e-05 rpy=0.0 -0.0 0.0 -> xyz=0.039132 -0.000136 -6e-05 rpy=0.0 -0.0 0.0
- joint finger_1_fingertip_1_DIP_Joint: axis -0.390731 0.920505 -0.0 -> 0.0 1.0 -0.0; origin xyz=0.028369 0.007387 -5e-06 rpy=0.0 -0.0 0.0 -> xyz=0.029 -0.004285 -5e-06 rpy=0.0 -0.0 0.0
- joint finger_2_distal_phalanx_1_PIP_Joint: axis -0.515038 0.857167 -0.0 -> 0.0 1.0 -0.0; origin xyz=0.033613 0.020039 -6e-05 rpy=0.0 -0.0 0.0 -> xyz=0.039132 -0.000135 -6e-05 rpy=0.0 -0.0 0.0
- joint finger_2_fingertip_1_DIP_Joint: axis -0.515038 0.857167 -0.0 -> 0.0 1.0 -0.0; origin xyz=0.027065 0.011263 -5e-06 rpy=0.0 -0.0 0.0 -> xyz=0.029 -0.004285 -5e-06 rpy=0.0 -0.0 0.0
- joint finger_3_distal_phalanx_1_PIP_Joint: axis -0.587785 0.809017 0.0 -> 0.0 1.0 -0.0; origin xyz=0.031738 0.022892 -6e-05 rpy=0.0 -0.0 0.0 -> xyz=0.039132 -0.000136 -6e-05 rpy=0.0 -0.0 0.0
- joint finger_3_fingertip_1_DIP_Joint: axis -0.587785 0.809017 -0.0 -> 0.0 1.0 -0.0; origin xyz=0.02598 0.013579 -5e-06 rpy=0.0 -0.0 0.0 -> xyz=0.029 -0.004285 -5e-06 rpy=0.0 -0.0 0.0
- joint finger_4_distal_phalanx_1_PIP_Joint: axis -0.587785 0.809017 0.0 -> 0.011122 0.999938 0.0; origin xyz=0.031738 0.022892 -6e-05 rpy=0.0 -0.0 0.0 -> xyz=0.039125 -0.000571 -0.00052 rpy=0.0 -0.0 0.0
- joint finger_4_fingertip_1_DIP_Joint: axis -0.587785 0.809017 -0.0 -> 0.011122 0.999938 -0.0; origin xyz=0.02598 0.013579 -5e-06 rpy=0.0 -0.0 0.0 -> xyz=0.028948 -0.004607 -0.000346 rpy=0.0 -0.0 0.0
- joint mmhand_thumb_1_finger_7_distal_phalanx_1_PIP_Joint: axis 0.862725 0.240955 0.444574 -> 0.745353 -0.666627 -0.00761; origin xyz=0.019099 -0.007442 -0.033335 rpy=0.0 -0.0 0.0 -> xyz=-0.007367 -0.007604 -0.037673 rpy=0.0 -0.0 0.0
- joint mmhand_thumb_1_finger_7_fingertip_1_DIP_Joint: axis 0.862725 0.240955 0.444574 -> 0.745353 -0.666627 -0.00761; origin xyz=0.010549 -0.006561 -0.026553 rpy=0.0 -0.0 0.0 -> xyz=-0.008604 -0.002874 -0.027876 rpy=0.0 -0.0 0.0
- joint palm_1_finger_base_1_fixed_joint: origin xyz=-0.1039 0.040332 0.023697 rpy=0.0 -0.0 0.0 -> xyz=-0.103901 0.040332 0.023697 rpy=0.0 -0.0 0.0
- joint palm_1_finger_base_2_fixed_joint: origin xyz=-0.1036 0.064332 0.023697 rpy=0.0 -0.0 0.0 -> xyz=-0.103901 0.064632 0.023697 rpy=0.0 -0.0 0.0
- joint palm_1_finger_base_3_fixed_joint: origin xyz=-0.1039 0.088332 0.023697 rpy=0.0 -0.0 0.0 -> xyz=-0.103901 0.088332 0.023697 rpy=0.0 -0.0 0.0

Commit message: aug manip success

File: assets/mmhand/urdf/hand.urdf (robot description, URDF)
Before this commit: robot mmhand, 32 links, 31 joints
Joints:
- joint Thumb_CMC: limit lower=0.7 upper=1.51 effort=100 velocity=100 -> lower=0.0 upper=1.51 effort=100 velocity=100
- joint Thumb_MCP_AA: limit lower=-1.2 upper=0.07 effort=100 velocity=100 -> lower=-1.2 upper=1 effort=100 velocity=100

File: teleop_maniskill/assets/robot/nero_capture_mmhand.urdf (robot description, URDF)
Before this commit: robot nero_capture_mmhand, 42 links, 41 joints
Joints:
- joint Thumb_CMC: limit lower=0.0 upper=1.343904 effort=100 velocity=100 -> lower=0.0 upper=1.51 effort=100 velocity=100
- joint Thumb_MCP_AA: limit lower=0.0 upper=0.994838 effort=100 velocity=100 -> lower=-1.2 upper=1 effort=100 velocity=100

File: teleop_maniskill/assets/standalone_nero_mmhand.urdf (robot description, URDF)
Before this commit: robot standalone_nero_capture_mmhand, 42 links, 41 joints
Joints:
- joint Thumb_CMC: limit lower=0.0 upper=1.343904 effort=100 velocity=100 -> lower=0.0 upper=1.51 effort=100 velocity=100
- joint Thumb_MCP_AA: limit lower=0.0 upper=0.994838 effort=100 velocity=100 -> lower=-1.2 upper=1 effort=100 velocity=100

Commit message: fix: align thumb and robot fingertip pads

File: assets/mmhand/urdf/hand.urdf (robot description, URDF)
Before this commit: robot (Unsaved), 32 links, 31 joints
Joints:
- joint 1-tip: origin xyz=0.023001459 0.010424364 -0.004367931 rpy=0 0 0 -> xyz=0.01536449 0.004452079 -0.008175908 rpy=0 0 0
- joint 2-tip: origin xyz=0.021343147 0.013505685 -0.004311705 rpy=0 0 0 -> xyz=0.015364505 0.004452078 -0.008175907 rpy=0 0 0
- joint 3-tip: origin xyz=0.020106421 0.015325961 -0.004336191 rpy=0 0 0 -> xyz=0.01536449 0.004452078 -0.008175908 rpy=0 0 0
- joint 4-tip: origin xyz=0.020105907 0.015325727 -0.004336522 rpy=0 0 0 -> xyz=0.015315325 0.004282186 -0.008356225 rpy=0 0 0
- joint 5-tip: origin xyz=0.012366569 -0.000590601 -0.022397383 rpy=0 0 0 -> xyz=0.006628915 -0.000976518 -0.017136225 rpy=1.531486234 -0.730633954 -0.704777306
